File: weatherStationv3.kicad_pcb (KiCad board)
At the start: 2 copper layers, 95 x 73 mm, 53 parts, among them J1 5-16V, J10 ANTENNA, J11 RS485_TERM, J2 USB_PWR_IN, J3 PORT1, J4 PORT2, J5 PORT3, J6 PORT4, J7 3.3-5V, J8 I2C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

Commit message: changeport connectors, move lora module, and impedance-match antenna
Parts:
- J3, J4, J5, J6: footprint Connector_Molex:Molex_KK-254_AE-6410-06A_1x06_P2.54mm_Vertical -> Connector_JST:JST_XH_B5B-XH-A_1x05_P2.50mm_Vertical
- moved C10 24.7 mm to (74.1, 83.8), turned to 90 degrees
- moved C6 13.0 mm to (78.6, 79.1)
- moved U4 12.5 mm to (90.1, 78.6)
- moved R3 0.75 mm to (97.3, 113.4)
- moved R4 0.75 mm to (107.4, 116.9)
Routing:
- net Net-(J10-In): track 23.0 -> 10.5 mm
- net /SCK: track 16.2 -> 28.5 mm
- net /MISO: track 15.6 -> 27.2 mm, vias 0 -> 2
- net /LORA_RESET: track 15.2 -> 24.9 mm
- net /LORA_CS: track 14.9 -> 24.5 mm
- net /MOSI: track 30.6 -> 36.8 mm
- net /LORA_DIO0: track 28.8 -> 34.0 mm
- net /LORA_DIO1: track 28.5 -> 33.7 mm
- net /LORA_DIO2: track 28.2 -> 33.4 mm
- net GND: track 81.3 -> 77.4 mm, vias 9 -> 20
- net +3.3V: track 18.7 -> 15.7 mm
- net +5V: track 208.7 -> 206.3 mm
- net Net-(J1-Pin_2): track 9.98 -> 10.7 mm
- net /WAKEUP_EXT: track 136.5 -> 135.9 mm
- added copper zone on F.Cu, net GND
