File: ws1-basestation-pcb.kicad_pcb (KiCad board)
At the start: 2 copper layers, 95 x 73 mm, 53 parts, among them J1 5-16V, J10 ANTENNA, J11 RS485_TERM, J2 USB_PWR_IN, J3 PORT1, J4 PORT2, J5 PORT3, J6 PORT4, J7 3.3-5V, J8 I2C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

Commit message: rename project files
Parts:
- removed D4, D5: SMAJ5.0A, Diode_SMD:D_SMA
- moved D3 15.6 mm to (146.9, 68.6)
- moved J3 1.36 mm to (102.9, 61.6)
- moved J4 1.26 mm to (119.1, 61.6)
- moved J5 1.14 mm to (135.4, 61.6)
- moved J6 1.12 mm to (151.7, 61.6)
- moved R8 0.70 mm to (146.1, 100.2)
Routing:
- net /RS485_A: track 119.7 -> 103.6 mm, vias 3 -> 4
- net GND: track 77.4 -> 72.5 mm, vias 20 -> 18
- net +5V: track 206.3 -> 202.0 mm
- net /WAKEUP_EXT: track 135.9 -> 138.1 mm
- net /RS485_B: track 116.3 -> 118.4 mm, vias 3 -> 5
Other:
- board text added: "I²C"
- board text added: "UART"
