File: ws1-basestation-pcb.kicad_sch (KiCad schematic)
At the start: 52 parts, among them J1 5-16V, J10 ANTENNA, J11 RS485_TERM, J2 USB_PWR_IN, J3 PORT1, J4 PORT2, J5 PORT3, J6 PORT4, J7 3.3-5V, J8 I2C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

Commit message: rename project files
Parts:
- removed D4, D5: SMAJ5.0A, Diode_SMD:D_SMA, symbol Diode:SMAJ5.0A
